File: TPO_Potencia.sch (KiCad schematic (older format))
At the start: 30 parts

Commit message: Agrego varios footprints, los que faltan los aclaro en el ReadMe
Parts:
- C1: renamed from C?; footprint (none) -> Capacitor_SMD:C_0805_2012Metric
- C2: renamed from C?; value 100µF -> 2200µF
- C4, C5: renamed from C?; footprint (none) -> Capacitor_SMD:C_1210_3225Metric
- C6: renamed from C?; footprint (none) -> Capacitor_THT:C_Rect_L26.5mm_W8.5mm_P22.50mm_MKS4
- D1: renamed from D?; value 1N47xxA -> 1N4738(8,2v)
- D2: renamed from D?; footprint (none) -> Diode_THT:RBV25
- D3: renamed from D?; footprint (none) -> Diode_THT:Diode_Bridge_Round_D9.0mm
- D5, D6: renamed from D?; value 1N47xxA -> 1N4742A
- J1, J4: renamed from J?; footprint (none) -> TerminalBlock:TerminalBlock_Altech_AK300-2_P5.00mm
- J2: renamed from J?; value Entrada_Alterna -> Entrada 220V Trafo; footprint (none) -> TerminalBlock:TerminalBlock_Altech_AK300-2_P5.00mm
- J3: renamed from J?; value Entrada_Alterna -> Salida 12V alt; footprint (none) -> TerminalBlock:TerminalBlock_Altech_AK300-2_P5.00mm
- J5: renamed from J?; footprint (none) -> Connector_PinHeader_2.54mm:PinHeader_2x03_P2.54mm_Vertical
- L1: renamed from L?; footprint (none) -> TerminalBlock:TerminalBlock_Altech_AK300-2_P5.00mm
- L2: renamed from L?; footprint (none) -> TerminalBlock:TerminalBlock_Altech_AK300-3_P5.00mm
- R1: renamed from R?; value R -> 220; footprint (none) -> Resistor_SMD:R_0805_2012Metric
- R2, R3, R4, R5: renamed from R?; footprint (none) -> Resistor_SMD:R_0805_2012Metric
- U1: renamed from U?; footprint (none) -> Package_TO_SOT_SMD:SOT-323_SC-70
- U2: renamed from U?; footprint (none) -> Package_SO:SOIC-8_3.9x4.9mm_P1.27mm
- U3, U4: renamed from U?; footprint (none) -> Package_TO_SOT_THT:TO-220-3_Horizontal_TabDown
- gave numbers to parts that had none: 4

Commit message: IR2153 corregido
Connections:
- net at U2.8 (VB): now also C3.1, D4.1 (K)
Other:
- moved on the sheet: D4
Changed lines of the file:
@@
 L Diode:BA159 D4
 U 1 1 5F3006C3
-P 6000 3900
-F 0 "D4" H 6000 3683 50  0000 C CNN
-F 1 "BA159" H 6000 3774 50  0000 C CNN
-F 2 "Diode_THT:D_DO-41_SOD81_P10.16mm_Horizontal" H 6000 3725 50  0001 C CNN
-F 3 "http://diotec.com/tl_files/diotec/files/pdf/datasheets/ba157" H 6000 3900 50  0001 C CNN
-	1    6000 3900
+P 5850 3900
+F 0 "D4" H 5850 3683 50  0000 C CNN
+F 1 "BA159" H 5850 3774 50  0000 C CNN
+F 2 "Diode_THT:D_DO-41_SOD81_P10.16mm_Horizontal" H 5850 3725 50  0001 C CNN
+F 3 "http://diotec.com/tl_files/diotec/files/pdf/datasheets/ba157" H 5850 3900 50  0001 C CNN
+	1    5850 3900
 	-1   0    0    1
 $EndComp
@@
 Wire Wire Line
 	6300 4950 7250 4950
-Wire Wire Line
-	5500 4250 5500 3900
-Wire Wire Line
-	5500 3900 5850 3900
-Wire Wire Line
-	6150 3900 6300 3900
-Connection ~ 5500 3900
-Wire Wire Line
-	5500 3900 5500 3700
 $Comp
 L power:VCC #PWR0106
@@
 Wire Notes Line
 	1300 4600 3450 4600
+Wire Wire Line
+	5500 3700 5500 3900
+Wire Wire Line
+	5700 3900 5500 3900
+Connection ~ 5500 3900
+Wire Wire Line
+	5500 3900 5500 4250
+Wire Wire Line
+	6000 3900 6100 3900
+Wire Wire Line
+	6100 3900 6100 4450
+Wire Wire Line
+	5800 4450 6100 4450
+Connection ~ 6100 3900
+Wire Wire Line
+	6100 3900 6300 3900
 $EndSCHEMATC

Commit message: PCB terminado
Parts:
- removed D3: RBV3500, Diode_THT:Diode_Bridge_Round_D9.0mm, symbol Diode_Bridge:RBV3500
- added U5: DB153, Diode_THT:Diode_Bridge_DIP-4_W7.62mm_P5.08mm, symbol TPO_Potencia-rescue:W02M
- C1: footprint Capacitor_SMD:C_0805_2012Metric -> Capacitor_SMD:C_0805_2012Metric_Pad1.15x1.40mm_HandSolder; symbol Device:C -> TPO_Potencia-rescue:C-Device
- C2: value 2200µF -> 2200µF 25V/35V; footprint (none) -> Capacitor_THT:C_Radial_D16.0mm_H25.0mm_P7.50mm; symbol Device:CP -> TPO_Potencia-rescue:CP-Device
- C3: value 100µF -> 100µF 16V; footprint (none) -> Capacitor_THT:C_Radial_D5.0mm_H11.0mm_P2.00mm; symbol Device:CP -> TPO_Potencia-rescue:CP-Device
- C4, C5, C6: symbol Device:C -> TPO_Potencia-rescue:C-Device
- D1, D5, D6: symbol Diode:1N47xxA -> TPO_Potencia-rescue:1N47xxA-Diode
- D2: symbol Diode_Bridge:RBV3500 -> TPO_Potencia-rescue:RBV3500-Diode_Bridge
- D4: symbol Diode:BA159 -> TPO_Potencia-rescue:BA159-Diode
- J1, J2, J3, J4: symbol Connector:Screw_Terminal_01x02 -> TPO_Potencia-rescue:Screw_Terminal_01x02-Connector
- J5: symbol Connector_Generic:Conn_02x03_Odd_Even -> TPO_Potencia-rescue:Conn_02x03_Odd_Even-Connector_Generic
- L1: symbol pspice:INDUCTOR -> TPO_Potencia-rescue:INDUCTOR-pspice
- L2: footprint TerminalBlock:TerminalBlock_Altech_AK300-3_P5.00mm -> TerminalBlock:TerminalBlock_Altech_AK300-2_P5.00mm; symbol pspice:INDUCTOR -> TPO_Potencia-rescue:INDUCTOR-pspice
- R1, R2, R3, R4, R5: symbol Device:R -> TPO_Potencia-rescue:R-Device
- RV1: footprint (none) -> Potentiometer_THT:Potentiometer_Bourns_3296W_Vertical; symbol Device:R_POT -> TPO_Potencia-rescue:R_POT-Device
- SW1: footprint (none) -> Button_Switch_THT:SW_Slide_1P2T_CK_OS102011MS2Q; symbol Switch:SW_DIP_x01 -> TPO_Potencia-rescue:SW_DIP_x01-Switch
- U1: symbol Transistor_FET:SSM3K16FU -> TPO_Potencia-rescue:SSM3K16FU-Transistor_FET
- U2: symbol Driver_FET:IR2153 -> TPO_Potencia-rescue:IR2153-Driver_FET
- U3, U4: footprint Package_TO_SOT_THT:TO-220-3_Horizontal_TabDown -> Package_TO_SOT_THT:TO-220-3_Vertical; symbol Transistor_FET:STP12N50M2 -> TPO_Potencia-rescue:STP12N50M2-Transistor_FET
Connections:
- net GND: now also U5.2 (-)
- net V1_alt_12V: now also U5.4 (~~)
- net V2_alt_12V: now also U5.3 (~~)
- net at D2.2 (~~), J1.1 (Pin_1): now also J2.2 (Pin_2); no longer J2.1 (Pin_1)
- net at D2.3 (~~), J1.2 (Pin_2): now also J2.1 (Pin_1); no longer J2.2 (Pin_2)
- net at J4.2 (Pin_2): now also J5.5 (Pin_5); no longer J5.1 (Pin_1)
- net at C2.1: now also J5.1 (Pin_1), U5.1 (+); no longer J5.5 (Pin_5)
Other:
- moved on the sheet: C2, J4
